File: robotont-motor-board.sch (KiCad schematic (older format))
At the start: 28 parts, among them J1 PWR_IN, J2 ENC, J3 MOTOR, J4 Conn_02x05_Odd_Even, U1 DMS3015SSS-13, U3 MIC5205-X.X

Commit message: v2.1 with jlcpcb components
Parts:
- removed SI8652: SI8652-IS, Package_SO:SOIC-16_3.9x9.9mm_P1.27mm, symbol robotont-motor-board:SI8452-IS
- removed U1: DMS3015SSS-13, Package_SO:SOIC-8-1EP_3.9x4.9mm_P1.27mm_EP2.29x3mm, symbol robotont-motor-board-eagle-import:DMS3015SSS-13
- added H1, H2: MountingHole_Pad, MountingHole:MountingHole_3mm_Pad, symbol Mechanical:MountingHole_Pad
- added U1: NTMS4807N, Package_SO:SO-8_3.9x4.9mm_P1.27mm, symbol robotont-motor-board:NTMS4807N
- added U2: Si8641BD-B-IS, Package_SO:SOIC-16W_7.5x10.3mm_P1.27mm, symbol Isolator:Si8641BD-B-IS
- C1, C2, C6, C8, C9: LCSC # (none) -> C14663
- C3: LCSC # (none) -> C21117
- C5, C7: LCSC # (none) -> C13585
- D1: LCSC # (none) -> C115273
- D2: LCSC # (none) -> C72043
- F1: Field4 C182976 -> (none); LCSC # (none) -> C182976
- J1: footprint Connector_AMASS:AMASS_XT30PW-M_1x02_P2.50mm_Horizontal -> robotont-motor-board:KF2510-2AWG
- J4: footprint footprints:CONN-TE-MICROMATCH-10X2-PTH -> footprints:CONN-TE-MICROMATCH-5X2-PTH-BOSS
- R1: LCSC # (none) -> C25803
- R2: LCSC # (none) -> C22775
- R3, R7: LCSC # (none) -> C25804
- R4: LCSC # (none) -> C4190
- R5, R6: LCSC # (none) -> C23204
- U3: LCSC # (none) -> C70431
Connections:
- net labels added: FAULT_D, FB_D
- net labels removed: FB
- wire segments 143 -> 140
Other:
- note added: "Driver block"
- note added: "Input regulation"
- note added: "Mounting holes"
- moved on the sheet: C1, C10, C2, C3, C4, C5, C6, C7, C8, C9, D1, D2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
